Commit message: added dampeners

File: quad2.xacro (robot description, xacro)
@@ -124,13 +124,13 @@
 <link name="back_right_lower">
     <visual>
-    <origin rpy="0 0 0" xyz="0 0 -0.05"/>
-      <geometry>
-        <cylinder length="0.1" radius="0.005"/>
-      </geometry>
-    </visual>
-    <collision>
-    <origin rpy="0 0 0" xyz="0 0 -0.05"/>
-      <geometry>
-        <cylinder length="0.1" radius="0.005"/>
+    <origin rpy="0 0 0" xyz="0 0 -0.035"/>
+      <geometry>
+        <cylinder length="0.07" radius="0.005"/>
+      </geometry>
+    </visual>
+    <collision>
+    <origin rpy="0 0 0" xyz="0 0 -0.035"/>
+      <geometry>
+        <cylinder length="0.07" radius="0.005"/>
       </geometry>
     </collision>
@@ -148,9 +148,34 @@
     <joint_properties damping="0.0" friction="0.05"/>
   </joint>
+<link name="back_right_dampener">
+    <visual>
+    <origin rpy="0 0 0" xyz="0 0 -0.05"/>
+      <geometry>
+        <cylinder length="0.025" radius="0.006"/>
+      </geometry>
+    </visual>
+    <collision>
+    <origin rpy="0 0 0" xyz="0 0 -0.05"/>
+      <geometry>
+        <cylinder length="0.025" radius="0.006"/>
+      </geometry>
+    </collision>
+    <inertial>
+      <mass value="0.025"/>
+      <inertia ixx="1.05e-4" ixy="0.0" ixz="0.0" iyy="0.0" iyz="0.0" izz="1.05e-4"/>
+    </inertial>
+  </link>
+  <joint name="back_right_damp_joint" type="prismatic">
+    <axis xyz="0 0 1"/>
+    <parent link="back_right_lower"/>
+    <child link="back_right_dampener"/>
+    <origin rpy="0 0 0" xyz="0 0 -0.035"/>
+    <limit lower="0.0" upper="0.025" />
+  </joint>
   <link name="back_right_foot">
     <visual>
     <origin rpy="0 0 0" xyz="0 0 0"/>
       <geometry>
-        <sphere radius="0.006"/>
+        <sphere radius="0.007"/>
       </geometry>
     </visual>
@@ -158,5 +183,5 @@
     <origin rpy="0 0 0" xyz="0 0 0"/>
       <geometry>
-        <sphere radius="0.006"/>
+        <sphere radius="0.007"/>
       </geometry>
     </collision>
@@ -167,7 +192,7 @@
   </link>
   <joint name="back_right_sensor" type="fixed">
-    <parent link="back_right_lower"/>
+    <parent link="back_right_dampener"/>
     <child link="back_right_foot"/>
-    <origin rpy="0 0 0" xyz="0 0 -0.1"/>
+    <origin rpy="0 0 0" xyz="0 0 -0.063"/>
     <joint_properties damping="0.0" friction="0.05"/>
   </joint>
@@ -252,13 +277,13 @@
 <link name="front_right_lower">
     <visual>
-    <origin rpy="0 0 0" xyz="0 0 -0.05"/>
-      <geometry>
-        <cylinder length="0.1" radius="0.005"/>
-      </geometry>
-    </visual>
-    <collision>
-    <origin rpy="0 0 0" xyz="0 0 -0.05"/>
-      <geometry>
-        <cylinder length="0.1" radius="0.005"/>
+    <origin rpy="0 0 0" xyz="0 0 -0.035"/>
+      <geometry>
+        <cylinder length="0.07" radius="0.005"/>
+      </geometry>
+    </visual>
+    <collision>
+    <origin rpy="0 0 0" xyz="0 0 -0.035"/>
+      <geometry>
+        <cylinder length="0.07" radius="0.005"/>
       </geometry>
     </collision>
@@ -276,9 +301,34 @@
     <joint_properties damping="0.0" friction="0.05"/>
   </joint>
+<link name="front_right_dampener">
+    <visual>
+    <origin rpy="0 0 0" xyz="0 0 -0.05"/>
+      <geometry>
+        <cylinder length="0.025" radius="0.006"/>
+      </geometry>
+    </visual>
+    <collision>
+    <origin rpy="0 0 0" xyz="0 0 -0.05"/>
+      <geometry>
+        <cylinder length="0.025" radius="0.006"/>
+      </geometry>
+    </collision>
+    <inertial>
+      <mass value="0.025"/>
+      <inertia ixx="1.05e-4" ixy="0.0" ixz="0.0" iyy="0.0" iyz="0.0" izz="1.05e-4"/>
+    </inertial>
+  </link>
+  <joint name="front_right_damp_joint" type="prismatic">
+    <axis xyz="0 0 1"/>
+    <parent link="front_right_lower"/>
+    <child link="front_right_dampener"/>
+    <origin rpy="0 0 0" xyz="0 0 -0.035"/>
+    <limit  lower="0.0" upper="0.025" />
+  </joint>
   <link name="front_right_foot">
     <visual>
     <origin rpy="0 0 0" xyz="0 0 0"/>
       <geometry>
-        <sphere radius="0.006"/>
+        <sphere radius="0.007"/>
       </geometry>
     </visual>
@@ -286,5 +336,5 @@
     <origin rpy="0 0 0" xyz="0 0 0"/>
       <geometry>
-        <sphere radius="0.006"/>
+        <sphere radius="0.007"/>
       </geometry>
     </collision>
@@ -295,7 +345,7 @@
   </link>
   <joint name="front_right_sensor" type="fixed">
-    <parent link="front_right_lower"/>
+    <parent link="front_right_dampener"/>
     <child link="front_right_foot"/>
-    <origin rpy="0 0 0" xyz="0 0 -0.1"/>
+    <origin rpy="0 0 0" xyz="0 0 -0.063"/>
     <joint_properties damping="0.0" friction="0.05"/>
   </joint>
@@ -380,13 +430,13 @@
 <link name="back_left_lower">
     <visual>
-    <origin rpy="0 0 0" xyz="0 0 -0.05"/>
-      <geometry>
-        <cylinder length="0.1" radius="0.005"/>
-      </geometry>
-    </visual>
-    <collision>
-    <origin rpy="0 0 0" xyz="0 0 -0.05"/>
-      <geometry>
-        <cylinder length="0.1" radius="0.005"/>
+    <origin rpy="0 0 0" xyz="0 0 -0.035"/>
+      <geometry>
+        <cylinder length="0.07" radius="0.005"/>
+      </geometry>
+    </visual>
+    <collision>
+    <origin rpy="0 0 0" xyz="0 0 -0.035"/>
+      <geometry>
+        <cylinder length="0.07" radius="0.005"/>
       </geometry>
     </collision>
@@ -404,9 +454,34 @@
     <joint_properties damping="0.0" friction="0.05"/>
   </joint>
+<link name="back_left_dampener">
+    <visual>
+    <origin rpy="0 0 0" xyz="0 0 -0.05"/>
+      <geometry>
+        <cylinder length="0.025" radius="0.006"/>
+      </geometry>
+    </visual>
+    <collision>
+    <origin rpy="0 0 0" xyz="0 0 -0.05"/>
+      <geometry>
+        <cylinder length="0.025" radius="0.006"/>
+      </geometry>
+    </collision>
+    <inertial>
+      <mass value="0.025"/>
+      <inertia ixx="1.05e-4" ixy="0.0" ixz="0.0" iyy="0.0" iyz="0.0" izz="1.05e-4"/>
+    </inertial>
+  </link>
+  <joint name="back_left_damp_joint" type="prismatic">
+    <axis xyz="0 0 1"/>
+    <parent link="back_left_lower"/>
+    <child link="back_left_dampener"/>
+    <origin rpy="0 0 0" xyz="0 0 -0.035"/>
+    <limit  lower="0.0" upper="0.025" />
+  </joint>
 <link name="back_left_foot">
     <visual>
     <origin rpy="0 0 0" xyz="0 0 0"/>
       <geometry>
-        <sphere radius="0.006"/>
+        <sphere radius="0.007"/>
       </geometry>
     </visual>
@@ -414,5 +489,5 @@
     <origin rpy="0 0 0" xyz="0 0 0"/>
       <geometry>
-        <sphere radius="0.006"/>
+        <sphere radius="0.007"/>
       </geometry>
     </collision>
@@ -423,7 +498,7 @@
   </link>
    <joint name="back_left_sensor" type="fixed">
-    <parent link="back_left_lower"/>
+    <parent link="back_left_dampener"/>
     <child link="back_left_foot"/>
-    <origin rpy="0 0 0" xyz="0 0 -0.1"/>
+    <origin rpy="0 0 0" xyz="0 0 -0.063"/>
     <joint_properties damping="0.0" friction="0.05"/>
   </joint>
@@ -508,13 +583,13 @@
 <link name="front_left_lower">
     <visual>
-    <origin rpy="0 0 0" xyz="0 0 -0.05"/>
-      <geometry>
-        <cylinder length="0.1" radius="0.005"/>
-      </geometry>
-    </visual>
-    <collision>
-    <origin rpy="0 0 0" xyz="0 0 -0.05"/>
-      <geometry>
-        <cylinder length="0.1" radius="0.005"/>
+    <origin rpy="0 0 0" xyz="0 0 -0.035"/>
+      <geometry>
+        <cylinder length="0.07" radius="0.005"/>
+      </geometry>
+    </visual>
+    <collision>
+    <origin rpy="0 0 0" xyz="0 0 -0.035"/>
+      <geometry>
+        <cylinder length="0.07" radius="0.005"/>
       </geometry>
     </collision>
@@ -532,9 +607,34 @@
     <joint_properties damping="0.0" friction="0.05"/>
   </joint>
+<link name="front_left_dampener">
+    <visual>
+    <origin rpy="0 0 0" xyz="0 0 -0.05"/>
+      <geometry>
+        <cylinder length="0.025" radius="0.006"/>
+      </geometry>
+    </visual>
+    <collision>
+    <origin rpy="0 0 0" xyz="0 0 -0.05"/>
+      <geometry>
+        <cylinder length="0.025" radius="0.006"/>
+      </geometry>
+    </collision>
+    <inertial>
+      <mass value="0.025"/>
+      <inertia ixx="1.05e-4" ixy="0.0" ixz="0.0" iyy="0.0" iyz="0.0" izz="1.05e-4"/>
+    </inertial>
+  </link>
+  <joint name="front_left_damp_joint" type="prismatic">
+    <axis xyz="0 0 1"/>
+    <parent link="front_left_lower"/>
+    <child link="front_left_dampener"/>
+    <origin rpy="0 0 0" xyz="0 0 -0.035"/>
+    <limit  lower="0.0" upper="0.025" />
+  </joint>
 <link name="front_left_foot">
     <visual>
     <origin rpy="0 0 0" xyz="0 0 0"/>
       <geometry>
-        <sphere radius="0.006"/>
+        <sphere radius="0.007"/>
       </geometry>
     </visual>
@@ -542,5 +642,5 @@
     <origin rpy="0 0 0" xyz="0 0 0"/>
       <geometry>
-        <sphere radius="0.006"/>
+        <sphere radius="0.007"/>
       </geometry>
     </collision>
@@ -551,7 +651,7 @@
   </link>
    <joint name="front_left_sensor" type="fixed">
-    <parent link="front_left_lower"/>
+    <parent link="front_left_dampener"/>
     <child link="front_left_foot"/>
-    <origin rpy="0 0 0" xyz="0 0 -0.1"/>
+    <origin rpy="0 0 0" xyz="0 0 -0.063"/>
     <joint_properties damping="0.0" friction="0.05"/>
   </joint>

Commit message: dwawing force

File: quad2.xacro (robot description, xacro)
@@ -15,5 +15,5 @@
     </collision>
     <inertial>
-      <mass value="2"/>
+      <mass value="3"/>
       <inertia ixx="0.01366667" ixy="0.0" ixz="0.0" iyy="0.01293333" iyz="0.0" izz="4.06666667e-3"/>
         <origin  xyz="0 0 0.32"/>
@@ -172,4 +172,5 @@
     <origin rpy="0 0 0" xyz="0 0 -0.035"/>
     <limit lower="0.0" upper="0.025" />
+    <joint_properties damping="0.05" friction="0.05"/>
   </joint>
   <link name="back_right_foot">
@@ -325,4 +326,5 @@
     <origin rpy="0 0 0" xyz="0 0 -0.035"/>
     <limit  lower="0.0" upper="0.025" />
+    <joint_properties damping="0.05" friction="0.05"/>
   </joint>
   <link name="front_right_foot">
@@ -478,4 +480,5 @@
     <origin rpy="0 0 0" xyz="0 0 -0.035"/>
     <limit  lower="0.0" upper="0.025" />
+    <joint_properties damping="0.05" friction="0.05"/>
   </joint>
 <link name="back_left_foot">
@@ -631,4 +634,5 @@
     <origin rpy="0 0 0" xyz="0 0 -0.035"/>
     <limit  lower="0.0" upper="0.025" />
+    <joint_properties damping="0.05" friction="0.05"/>
   </joint>
 <link name="front_left_foot">
