Commit message: balancing without shock dampening

File: resources/quad.xacro (robot description, xacro)
@@ -162,6 +162,6 @@
     </collision>
     <inertial>
-      <mass value="0.025"/>
-      <inertia ixx="4.166666666666667e-06" ixy="0.0" ixz="0.0" iyy="0.0" iyz="0.0" izz="4.166666666666667e-06"/>
+      <mass value="0.005"/>
+      <inertia ixx="8.32e-07" ixy="0.0" ixz="0.0" iyy="0.0" iyz="0.0" izz="8.32e-07"/>
     </inertial>
   </link>
@@ -172,5 +172,5 @@
     <origin rpy="0 0 0" xyz="0 0 -0.046"/>
     <limit  lower="0.0" upper="0.012" />
-    <joint_properties damping="0.05" friction="0.00"/>
+    <joint_properties damping="0.05" friction="0.1"/>
   </joint>
 <link name="back_right_foot">
@@ -188,6 +188,6 @@
     </collision>
     <inertial>
-      <mass value="0.025"/>
-      <inertia ixx="6.400000000000001e-07" ixy="0.0" ixz="0.0" iyy="6.400000000000001e-07" iyz="0.0" izz="6.400000000000001e-07"/>
+      <mass value="0.005"/>
+      <inertia ixx="1.28e-07" ixy="0.0" ixz="0.0" iyy="1.28e-07" iyz="0.0" izz="1.28e-07"/>
     </inertial>
   </link>
